File: eagle-cad/line_follower.sch (EAGLE design)
At the start: 16 parts

Commit message: fixed led resistor
Parts:
- added R1: 330, SparkFun-Passives:RESISTOREZ
- R3, R4: value 300K -> 330K
Connections:
- new net N$6: LED1.A, R1.1
- net GND: now also R1.2; no longer LED1.A
Changed lines of the file:
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@@
 <part name="10K" library="SparkFun-Passives" deviceset="POTENTIOMETER" device=""/>
 <part name="R2" library="SparkFun-Passives" deviceset="RESISTOR" device="EZ" value="1K"/>
-<part name="R3" library="SparkFun-Passives" deviceset="RESISTOR" device="EZ" value="300K"/>
-<part name="R4" library="SparkFun-Passives" deviceset="RESISTOR" device="EZ" value="300K"/>
+<part name="R3" library="SparkFun-Passives" deviceset="RESISTOR" device="EZ" value="330K"/>
+<part name="R4" library="SparkFun-Passives" deviceset="RESISTOR" device="EZ" value="330K"/>
 <part name="SCREW_TERMINAL" library="SparkFun-Connectors" deviceset="M02" device="JST-PTH-VERT"/>
 <part name="SW1" library="adafruit" deviceset="SWITCH_PUSHBUTTON" device="EVQ-PE"/>
@@
 <part name="C1" library="SparkFun-Capacitors" deviceset="CAP" device="EZ" value="0.1uF"/>
 <part name="C2" library="SparkFun-Capacitors" deviceset="CAP" device="EZ" value="0.1uF"/>
+<part name="R1" library="SparkFun-Passives" deviceset="RESISTOR" device="EZ" value="330"/>
 </parts>
 <sheets>
@@
 <instance part="C1" gate="G$1" x="5.08" y="66.04"/>
 <instance part="C2" gate="G$1" x="-27.94" y="66.04"/>
+<instance part="R1" gate="G$1" x="45.72" y="2.54" rot="R180"/>
 </instances>
 <busses>
@@
 <wire x1="-12.7" y1="48.26" x2="-40.64" y2="48.26" width="0.1524" layer="91"/>
 <junction x="-40.64" y="48.26"/>
-<pinref part="LED1" gate="G$1" pin="A"/>
-<wire x1="25.4" y1="2.54" x2="63.5" y2="2.54" width="0.1524" layer="91"/>
-<junction x="25.4" y="2.54"/>
 <pinref part="C2" gate="G$1" pin="2"/>
 <wire x1="-27.94" y1="63.5" x2="-27.94" y2="58.42" width="0.1524" layer="91"/>
@@
 <wire x1="5.08" y1="63.5" x2="5.08" y2="58.42" width="0.1524" layer="91"/>
 <junction x="5.08" y="58.42"/>
+<pinref part="R1" gate="G$1" pin="2"/>
+<wire x1="25.4" y1="2.54" x2="40.64" y2="2.54" width="0.1524" layer="91"/>
+<junction x="25.4" y="2.54"/>
 </segment>
 <segment>
@@
 </segment>
 </net>
+<net name="N$6" class="0">
+<segment>
+<pinref part="R1" gate="G$1" pin="1"/>
+<pinref part="LED1" gate="G$1" pin="A"/>
+<wire x1="50.8" y1="2.54" x2="63.5" y2="2.54" width="0.1524" layer="91"/>
+</segment>
+</net>

Commit message: fixed the motor power source
Connections:
- removed net 9V: C2.1, DRV8835.VIN, LM7805.IN, SCREW_TERMINAL.1
- net VDD: now also C2.1, DRV8835.VIN, LM7805.IN, SCREW_TERMINAL.1
Changed lines of the file:
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@@
-</segment>
-<segment>
-<pinref part="LM7805" gate="1" pin="OUT"/>
-<wire x1="-2.54" y1="76.2" x2="5.08" y2="76.2" width="0.1524" layer="91"/>
-<pinref part="DRV8835" gate="G$1" pin="VCC"/>
-<pinref part="C1" gate="G$1" pin="1"/>
-<wire x1="5.08" y1="76.2" x2="50.8" y2="76.2" width="0.1524" layer="91"/>
-<wire x1="5.08" y1="71.12" x2="5.08" y2="76.2" width="0.1524" layer="91"/>
-<junction x="5.08" y="76.2"/>
 </segment>
 <segment>
@@
 <wire x1="71.12" y1="2.54" x2="73.66" y2="2.54" width="0.1524" layer="91"/>
 <label x="73.66" y="2.54" size="1.778" layer="95" xref="yes"/>
+</segment>
+<segment>
+<pinref part="SCREW_TERMINAL" gate="G$1" pin="1"/>
+<pinref part="LM7805" gate="1" pin="IN"/>
+<wire x1="-27.94" y1="76.2" x2="-17.78" y2="76.2" width="0.1524" layer="91"/>
+<junction x="-27.94" y="76.2"/>
+<pinref part="C2" gate="G$1" pin="1"/>
+<wire x1="-27.94" y1="71.12" x2="-27.94" y2="76.2" width="0.1524" layer="91"/>
+<pinref part="SUPPLY1" gate="VDD" pin="VDD"/>
+<wire x1="-43.18" y1="88.9" x2="-43.18" y2="76.2" width="0.1524" layer="91"/>
+<wire x1="-43.18" y1="76.2" x2="-27.94" y2="76.2" width="0.1524" layer="91"/>
+<junction x="-43.18" y="76.2"/>
+<wire x1="-43.18" y1="76.2" x2="-45.72" y2="76.2" width="0.1524" layer="91"/>
+</segment>
+<segment>
+<pinref part="DRV8835" gate="G$1" pin="VIN"/>
+<wire x1="83.82" y1="76.2" x2="99.06" y2="76.2" width="0.1524" layer="91"/>
+<wire x1="99.06" y1="76.2" x2="99.06" y2="83.82" width="0.1524" layer="91"/>
+<pinref part="LM7805" gate="1" pin="OUT"/>
+<wire x1="-2.54" y1="76.2" x2="5.08" y2="76.2" width="0.1524" layer="91"/>
+<pinref part="DRV8835" gate="G$1" pin="VCC"/>
+<pinref part="C1" gate="G$1" pin="1"/>
+<wire x1="5.08" y1="76.2" x2="50.8" y2="76.2" width="0.1524" layer="91"/>
+<wire x1="5.08" y1="71.12" x2="5.08" y2="76.2" width="0.1524" layer="91"/>
+<junction x="5.08" y="76.2"/>
+<wire x1="99.06" y1="83.82" x2="5.08" y2="83.82" width="0.1524" layer="91"/>
+<wire x1="5.08" y1="83.82" x2="5.08" y2="76.2" width="0.1524" layer="91"/>
 </segment>
 </net>
@@
 </segment>
 </net>
-<net name="9V" class="0">
-<segment>
-<pinref part="SUPPLY1" gate="VDD" pin="VDD"/>
-<wire x1="-43.18" y1="88.9" x2="-43.18" y2="76.2" width="0.1524" layer="91"/>
-<pinref part="SCREW_TERMINAL" gate="G$1" pin="1"/>
-<wire x1="-43.18" y1="76.2" x2="-45.72" y2="76.2" width="0.1524" layer="91"/>
-<pinref part="LM7805" gate="1" pin="IN"/>
-<wire x1="-43.18" y1="76.2" x2="-27.94" y2="76.2" width="0.1524" layer="91"/>
-<junction x="-43.18" y="76.2"/>
-<pinref part="DRV8835" gate="G$1" pin="VIN"/>
-<wire x1="-27.94" y1="76.2" x2="-17.78" y2="76.2" width="0.1524" layer="91"/>
-<wire x1="83.82" y1="76.2" x2="99.06" y2="76.2" width="0.1524" layer="91"/>
-<wire x1="99.06" y1="76.2" x2="99.06" y2="83.82" width="0.1524" layer="91"/>
-<wire x1="99.06" y1="83.82" x2="-27.94" y2="83.82" width="0.1524" layer="91"/>
-<wire x1="-27.94" y1="83.82" x2="-27.94" y2="76.2" width="0.1524" layer="91"/>
-<junction x="-27.94" y="76.2"/>
-<pinref part="C2" gate="G$1" pin="1"/>
-<wire x1="-27.94" y1="71.12" x2="-27.94" y2="76.2" width="0.1524" layer="91"/>
-</segment>
-</net>
